File: SoftHRUF/Split Corded/Split Cordedv0.1.sch (KiCad schematic (older format))
At the start: 98 parts, among them CON1 AVR-ISP-6, P1 USB_B, P2 10p10c_LEFT, P3 10p10c_RIGHT, SW1 SW_PUSH, SW10 SW_PUSH, SW11 SW_PUSH, SW12 SW_PUSH, SW13 SW_PUSH, SW14 SW_PUSH, SW15 SW_PUSH, SW16 SW_PUSH, SW17 SW_PUSH, SW18 SW_PUSH, SW19 SW_PUSH, SW2 SW_PUSH, SW20 SW_PUSH, SW21 SW_PUSH, SW22 SW_PUSH, SW23 SW_PUSH, SW24 SW_PUSH, SW25 SW_PUSH, SW26 SW_PUSH, SW27 SW_PUSH, SW28 SW_PUSH, SW29 SW_PUSH, SW3 SW_PUSH, SW30 SW_PUSH, SW31 SW_PUSH, SW32 SW_PUSH, SW33 SW_PUSH, SW34 SW_PUSH, SW35 SW_PUSH, SW36 SW_PUSH, SW37 SW_PUSH, SW38 SW_PUSH, SW39 SW_PUSH, SW4 SW_PUSH, SW40 SW_PUSH, SW41 Switch_DPST, SW5 SW_PUSH, SW6 SW_PUSH, SW7 SW_PUSH, SW8 SW_PUSH, SW9 SW_PUSH, U1 IP4234CZ6, U2 ATmega32U4-AU, Y1 Crystal_Small

Commit message: In the middle of making last few changes. Last thing I need to do is fiddle with the USB connector, since the first one showed signs of weakness.
Parts:
- P1: symbol USB_A -> USB_A-RESCUE-Split_Cordedv0.1
- U2: symbol ATmega32U4-AU -> ATmega32U4-AU-RESCUE-Split_Cordedv0.1
Changed lines of the file:
@@
 EESchema Schematic File Version 2
+LIBS:Split Cordedv0.1-rescue
 LIBS:power
 LIBS:device
@@
 LIBS:contrib
 LIBS:valves
-LIBS:aker
-LIBS:atmega32u4
-LIBS:dtsjw
-LIBS:mx1a-simple
-LIBS:oupiin_usb
 LIBS:Split Cordedv0.1-cache
 EELAYER 25 0
@@
 $EndDescr
 $Comp
-L USB_A P1
+L USB_A-RESCUE-Split_Cordedv0.1 P1
 U 1 1 57FED16D
 P 5250 6400
@@
 $EndComp
 $Comp
-L ATmega32U4-AU U2
+L ATmega32U4-AU-RESCUE-Split_Cordedv0.1 U2
 U 1 1 57FED110
 P 3000 5800
